File: genoswitch-rp2040/genoswitch-rp2040.kicad_pcb (KiCad board)
At the start: 2 copper layers, 37 parts, among them J1 USB_B_Micro, J2 Conn_01x03_Socket-PicoDebug, J3 HW-SPI0, J4 HW-SPI1, J5 PIO-SPI0, J6 PIO-SPI1, J7 SERIAL, SW1 PTS815_SJM_250_SMTR_LFS, U1 NCP1117-3.3_SOT223, U2 W25Q128JVS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

Commit message: misc layout changes
Parts:
- moved C4 45.9 mm to (126.8, 66.3)
- moved H2 36.5 mm to (112.0, 58.9)
- moved J3 12.8 mm to (92.2, 46.8), turned to -90 degrees
- moved C15 8.83 mm to (127.0, 68.4)
- moved C6 8.83 mm to (126.2, 68.4)
- moved C8 8.83 mm to (128.9, 68.4)
- moved C10 8.83 mm to (129.6, 68.4)
- moved J5 1.79 mm to (92.2, 84.3)
Changed lines of the file:
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@@
   )
   (footprint "Capacitor_SMD:C_01005_0402Metric" (layer "F.Cu")
-    (at 138.39 68.321 90)
+    (at 129.562 68.4 90)
     (descr "Capacitor SMD 01005 (0402 Metric), square (rectangular) end terminal, IPC_7351 nominal, (Body size source: http://www.vishay.com/docs/20056/crcw01005e3.pdf), generated with kicad-footprint-generator")
     (tags "capacitor")
@@
   )
   (footprint "Capacitor_SMD:C_01005_0402Metric" (layer "F.Cu")
-    (at 135.05 68.325 90)
+    (at 126.222 68.404 90)
     (descr "Capacitor SMD 01005 (0402 Metric), square (rectangular) end terminal, IPC_7351 nominal, (Body size source: http://www.vishay.com/docs/20056/crcw01005e3.pdf), generated with kicad-footprint-generator")
     (tags "capacitor")
@@
   )
   (footprint "Capacitor_SMD:C_01005_0402Metric" (layer "F.Cu")
-    (at 135.812 68.325 -90)
+    (at 126.984 68.404 -90)
     (descr "Capacitor SMD 01005 (0402 Metric), square (rectangular) end terminal, IPC_7351 nominal, (Body size source: http://www.vishay.com/docs/20056/crcw01005e3.pdf), generated with kicad-footprint-generator")
     (tags "capacitor")
@@
   )
   (footprint "Connector_JST:JST_PH_S7B-PH-K_1x07_P2.00mm_Horizontal" (layer "F.Cu")
-    (at 93.89 84.805 -90)
+    (at 92.162 84.35 -90)
     (descr "JST PH series connector, S7B-PH-K (http://www.jst-mfg.com/product/pdf/eng/ePH.pdf), generated with kicad-footprint-generator")
     (tags "connector JST PH top entry")
@@
   )
   (footprint "Capacitor_SMD:C_01005_0402Metric" (layer "F.Cu")
-    (at 137.717 68.325 90)
+    (at 128.889 68.404 90)
     (descr "Capacitor SMD 01005 (0402 Metric), square (rectangular) end terminal, IPC_7351 nominal, (Body size source: http://www.vishay.com/docs/20056/crcw01005e3.pdf), generated with kicad-footprint-generator")
     (tags "capacitor")
@@
   )
   (footprint "MountingHole:MountingHole_2.7mm_M2.5" (layer "F.Cu")
-    (at 78.312 44.85 -90)
+    (at 112.012 58.85 -90)
     (descr "Mounting Hole 2.7mm, no annular, M2.5")
     (tags "mounting hole 2.7mm no annular m2.5")
@@
   )
   (footprint "Capacitor_SMD:C_01005_0402Metric" (layer "F.Cu")
-    (at 81.887 57)
+    (at 126.787 66.3)
     (descr "Capacitor SMD 01005 (0402 Metric), square (rectangular) end terminal, IPC_7351 nominal, (Body size source: http://www.vishay.com/docs/20056/crcw01005e3.pdf), generated with kicad-footprint-generator")
     (tags "capacitor")
@@
     (property "ki_keywords" "RP2040 ARM Cortex-M0+ USB")
     (attr smd)
-    (fp_text reference "U3" (at 26.338 -4.334) (layer "F.SilkS")
+    (fp_text reference "U3" (at 17.51 -4.255) (layer "F.SilkS")
         (effects (font (size 1 1) (thickness 0.15)))
     )
@@
   )
   (footprint "Connector_JST:JST_PH_S7B-PH-K_1x07_P2.00mm_Horizontal" (layer "F.Cu")
-    (at 87.592 58.77 90)
+    (at 92.162 46.8 -90)
     (descr "JST PH series connector, S7B-PH-K (http://www.jst-mfg.com/product/pdf/eng/ePH.pdf), generated with kicad-footprint-generator")
     (tags "connector JST PH top entry")
@@
     (fp_line (start 13.95 6.25) (end 13.95 -1.35)
       (stroke (width 0.1) (type solid)) (layer "F.Fab"))
-    (pad "1" thru_hole roundrect (at 0 0 90) (size 1.2 1.75) (drill 0.75) (layers "*.Cu" "*.Mask") (roundrect_rratio 0.208333)
+    (pad "1" thru_hole roundrect (at 0 0 270) (size 1.2 1.75) (drill 0.75) (layers "*.Cu" "*.Mask") (roundrect_rratio 0.208333)
       (net 5 "+3V3") (pinfunction "VDD") (pintype "passive"))
-    (pad "2" thru_hole oval (at 2 0 90) (size 1.2 1.75) (drill 0.75) (layers "*.Cu" "*.Mask")
+    (pad "2" thru_hole oval (at 2 0 270) (size 1.2 1.75) (drill 0.75) (layers "*.Cu" "*.Mask")
       (net 2 "GND") (pinfunction "GND") (pintype "passive"))
-    (pad "3" thru_hole oval (at 4 0 90) (size 1.2 1.75) (drill 0.75) (layers "*.Cu" "*.Mask")
+    (pad "3" thru_hole oval (at 4 0 270) (size 1.2 1.75) (drill 0.75) (layers "*.Cu" "*.Mask")
       (net 15 "/GPIO6") (pinfunction "CLK") (pintype "passive"))
-    (pad "4" thru_hole oval (at 6 0 90) (size 1.2 1.75) (drill 0.75) (layers "*.Cu" "*.Mask")
+    (pad "4" thru_hole oval (at 6 0 270) (size 1.2 1.75) (drill 0.75) (layers "*.Cu" "*.Mask")
       (net 16 "/GPIO4") (pinfunction "DOUT") (pintype "passive"))
-    (pad "5" thru_hole oval (at 8 0 90) (size 1.2 1.75) (drill 0.75) (layers "*.Cu" "*.Mask")
+    (pad "5" thru_hole oval (at 8 0 270) (size 1.2 1.75) (drill 0.75) (layers "*.Cu" "*.Mask")
       (net 17 "/GPIO7") (pinfunction "DIN") (pintype "passive"))
-    (pad "6" thru_hole oval (at 10 0 90) (size 1.2 1.75) (drill 0.75) (layers "*.Cu" "*.Mask")
+    (pad "6" thru_hole oval (at 10 0 270) (size 1.2 1.75) (drill 0.75) (layers "*.Cu" "*.Mask")
       (net 18 "/GPIO5") (pinfunction "CS") (pintype "passive"))
-    (pad "7" thru_hole oval (at 12 0 90) (size 1.2 1.75) (drill 0.75) (layers "*.Cu" "*.Mask")
+    (pad "7" thru_hole oval (at 12 0 270) (size 1.2 1.75) (drill 0.75) (layers "*.Cu" "*.Mask")
       (net 19 "/ADC_VREF") (pinfunction "VREF") (pintype "passive"))
     (model "${KICAD6_3DMODEL_DIR}/Connector_JST.3dshapes/JST_PH_S7B-PH-K_1x07_P2.00mm_Horizontal.wrl"
@@
   (gr_line (start 86.912 50.75) (end 131.662 50.75)
     (stroke (width 0.15) (type default)) (layer "User.1"))
-  (gr_line (start 103.312 44.25) (end 85.322 44.26)
+  (gr_line (start 107.012 44.25) (end 85.322 44.26)
     (stroke (width 0.15) (type default)) (layer "User.1"))
   (gr_line (start 85.322 44.26) (end 85.312 103.7)

Commit message: (ADC_CONN): Make GND pin 1
Parts:
- moved C15 10.5 mm to (137.4, 70.0)
- moved C6 10.5 mm to (136.6, 70.0)
- moved C10 10.5 mm to (139.9, 70.0)
- moved C4 10.5 mm to (137.2, 67.9)
- moved C8 10.5 mm to (139.3, 70.0)
- moved J5 3.61 mm to (92.4, 88.0)
- moved J6 1.95 mm to (122.2, 100.0)
- moved J3 0.25 mm to (92.4, 46.8)
Connections:
- J3 pad 1: +3V3 -> GND
- J3 pad 2: GND -> +3V3
- J4 pad 1: +3V3 -> GND
- J4 pad 2: GND -> +3V3
- J5 pad 1: +3V3 -> GND
- J5 pad 2: GND -> +3V3
- J6 pad 1: +3V3 -> GND
- J6 pad 2: GND -> +3V3
Other:
- board text added: "17.150mm"

Commit message: Reposition holes
Parts:
- moved H1 43.7 mm to (98.4, 47.5), turned to -90 degrees
- moved H2 32.5 mm to (114.1, 91.3), turned to 0 degrees
- moved J7 27.7 mm to (118.9, 64.2)
Changed lines of the file:
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@@
   )
   (footprint "MountingHole:MountingHole_2.7mm_M2.5" (layer "F.Cu")
-    (at 112.012 58.85 -90)
+    (at 114.062 91.3)
     (descr "Mounting Hole 2.7mm, no annular, M2.5")
     (tags "mounting hole 2.7mm no annular m2.5")
@@
     (property "ki_keywords" "mounting hole")
     (attr exclude_from_pos_files)
-    (fp_text reference "H2" (at 0 -3.7 90) (layer "F.SilkS")
-        (effects (font (size 1 1) (thickness 0.15)))
-    )
-    (fp_text value "M2.5" (at 0 3.7 90) (layer "F.Fab")
-        (effects (font (size 1 1) (thickness 0.15)))
-    )
-    (fp_text user "${REFERENCE}" (at 0 0 90) (layer "F.Fab")
+    (fp_text reference "H2" (at 0 -3.7) (layer "F.SilkS")
+        (effects (font (size 1 1) (thickness 0.15)))
+    )
+    (fp_text value "M2.5" (at 0 3.7) (layer "F.Fab")
+        (effects (font (size 1 1) (thickness 0.15)))
+    )
+    (fp_text user "${REFERENCE}" (at 0 0) (layer "F.Fab")
         (effects (font (size 1 1) (thickness 0.15)))
     )
@@
     (fp_circle (center 0 0) (end 2.95 0)
       (stroke (width 0.05) (type solid)) (fill none) (layer "F.CrtYd"))
-    (pad "" np_thru_hole circle (at 0 0 270) (size 2.7 2.7) (drill 2.7) (layers "F&B.Cu" "*.Mask"))
+    (pad "" np_thru_hole circle (at 0 0) (size 2.7 2.7) (drill 2.7) (layers "F&B.Cu" "*.Mask"))
   )
   (footprint "Resistor_SMD:R_01005_0402Metric" (layer "F.Cu")
@@
   )
   (footprint "MountingHole:MountingHole_2.7mm_M2.5" (layer "F.Cu")
-    (at 114.3 88.265)
+    (at 98.412 47.55 -90)
     (descr "Mounting Hole 2.7mm, no annular, M2.5")
     (tags "mounting hole 2.7mm no annular m2.5")
@@
     (property "ki_keywords" "mounting hole")
     (attr exclude_from_pos_files)
-    (fp_text reference "H1" (at 0 -3.7) (layer "F.SilkS")
-        (effects (font (size 1 1) (thickness 0.15)))
-    )
-    (fp_text value "M2.5" (at 0 3.7) (layer "F.Fab")
-        (effects (font (size 1 1) (thickness 0.15)))
-    )
-    (fp_text user "${REFERENCE}" (at 0 0) (layer "F.Fab")
+    (fp_text reference "H1" (at 0 -3.7 90) (layer "F.SilkS")
+        (effects (font (size 1 1) (thickness 0.15)))
+    )
+    (fp_text value "M2.5" (at 0 3.7 90) (layer "F.Fab")
+        (effects (font (size 1 1) (thickness 0.15)))
+    )
+    (fp_text user "${REFERENCE}" (at 0 0 90) (layer "F.Fab")
         (effects (font (size 1 1) (thickness 0.15)))
     )
@@
     (fp_circle (center 0 0) (end 2.95 0)
       (stroke (width 0.05) (type solid)) (fill none) (layer "F.CrtYd"))
-    (pad "" np_thru_hole circle (at 0 0) (size 2.7 2.7) (drill 2.7) (layers "*.Cu" "*.Mask"))
+    (pad "" np_thru_hole circle (at 0 0 270) (size 2.7 2.7) (drill 2.7) (layers "*.Cu" "*.Mask"))
   )
   (footprint "Resistor_SMD:R_01005_0402Metric" (layer "F.Cu")
@@
   )
   (footprint "Connector_PinHeader_2.54mm:PinHeader_1x02_P2.54mm_Vertical" (layer "F.Cu")
-    (at 97.227 46.93 90)
+    (at 118.937 64.15 90)
     (descr "Through hole straight pin header, 1x02, 2.54mm pitch, single row")
     (tags "Through hole pin header THT 1x02 2.54mm single row")
